Commit message: Add urdf and meshes in gz_sim package

File: src/gz_sim/urdf/nemo.urdf (robot description, URDF)
Before this commit: robot nemo, 13 links, 13 joints
Links:
- link l_foot_pitch: geometry collision mesh filename=package://gz_sim/meshes/nemo/l_foot_pitch.stl; visual mesh filename=package://gz_sim/meshes/nemo/l_foot_pitch.stl
- link l_foot_roll: geometry collision mesh filename=package://gz_sim/meshes/nemo/l_foot_roll.stl; visual mesh filename=package://gz_sim/meshes/nemo/l_foot_roll.stl
- link l_hip_pitch: geometry collision mesh filename=package://gz_sim/meshes/nemo/l_hip_pitch.stl; visual mesh filename=package://gz_sim/meshes/nemo/l_hip_pitch.stl
- link l_hip_roll: geometry collision mesh filename=package://gz_sim/meshes/nemo/l_hip_roll.stl; visual mesh filename=package://gz_sim/meshes/nemo/l_hip_roll.stl
- link l_hip_yaw: geometry collision mesh filename=package://gz_sim/meshes/nemo/l_hip_yaw.stl; visual mesh filename=package://gz_sim/meshes/nemo/l_hip_yaw.stl
- link l_knee: geometry collision mesh filename=package://gz_sim/meshes/nemo/l_knee.stl; visual mesh filename=package://gz_sim/meshes/nemo/l_knee.stl
- link pelvis: geometry collision mesh filename=package://gz_sim/meshes/nemo/pelvis_box.stl; visual mesh filename=package://gz_sim/meshes/nemo/pelvis_box.stl
- link r_foot_pitch: geometry collision mesh filename=package://gz_sim/meshes/nemo/r_foot_pitch.stl; visual mesh filename=package://gz_sim/meshes/nemo/r_foot_pitch.stl
- link r_foot_roll: geometry collision mesh filename=package://gz_sim/meshes/nemo/r_foot_roll.stl; visual mesh filename=package://gz_sim/meshes/nemo/r_foot_roll.stl
- link r_hip_pitch: geometry collision mesh filename=package://gz_sim/meshes/nemo/r_hip_pitch.stl; visual mesh filename=package://gz_sim/meshes/nemo/r_hip_pitch.stl
- link r_hip_roll: geometry collision mesh filename=package://gz_sim/meshes/nemo/r_hip_roll.stl; visual mesh filename=package://gz_sim/meshes/nemo/r_hip_roll.stl
- link r_hip_yaw: geometry collision mesh filename=package://gz_sim/meshes/nemo/r_hip_yaw.stl; visual mesh filename=package://gz_sim/meshes/nemo/r_hip_yaw.stl
- link r_knee: geometry collision mesh filename=package://gz_sim/meshes/nemo/r_knee.stl; visual mesh filename=package://gz_sim/meshes/nemo/r_knee.stl
Joints:
- removed joint floating_base
- removed joint l_foot_pitch
- removed joint l_foot_roll
- removed joint l_hip_pitch
- removed joint l_hip_roll
- removed joint l_hip_yaw
- removed joint l_knee
- removed joint r_foot_pitch
- removed joint r_foot_roll
- removed joint r_hip_pitch
- removed joint r_hip_roll
- removed joint r_hip_yaw
- removed joint r_knee
- added joint l_foot_pitch_joint: type revolute, parent l_knee, child l_foot_pitch, origin xyz=0 0.00635 -0.3366 rpy=0 0 0, axis 0 1 0, limit lower=-0.5 upper=0.5 effort=34.0 velocity=34.0
- added joint l_foot_roll_joint: type revolute, parent l_foot_pitch, child l_foot_roll, origin xyz=0.0889 0 0 rpy=0 0 0, axis 1 0 0, limit lower=-1.0 upper=1.0 effort=34.0 velocity=34.0
- added joint l_hip_pitch_joint: type revolute, parent pelvis, child l_hip_pitch, origin xyz=0 0.0762 0 rpy=0 0 0, axis 0 1 0, limit lower=-3.0 upper=3.0 effort=34.0 velocity=34.0
- added joint l_hip_roll_joint: type revolute, parent l_hip_pitch, child l_hip_roll, origin xyz=-0.05715 0.127 0 rpy=0 0 0, axis 1 0 0, limit lower=-0.279253 upper=1.0 effort=34.0 velocity=34.0
- added joint l_hip_yaw_joint: type revolute, parent l_hip_roll, child l_hip_yaw, origin xyz=0.06254 0 -0.1905 rpy=0 0 0, axis 0 0 1, limit lower=-2.5 upper=2.5 effort=34.0 velocity=34.0
- added joint l_knee_joint: type revolute, parent l_hip_yaw, child l_knee, origin xyz=0 0 -0.2286 rpy=0 0 0, axis 0 1 0, limit lower=-0.3 upper=2.0 effort=34.0 velocity=34.0
- added joint r_foot_pitch_joint: type revolute, parent r_knee, child r_foot_pitch, origin xyz=0 -0.00635 -0.3366 rpy=0 0 0, axis 0 1 0, limit lower=-0.5 upper=0.5 effort=34.0 velocity=34.0
- added joint r_foot_roll_joint: type revolute, parent r_foot_pitch, child r_foot_roll, origin xyz=0.0889 0 0 rpy=0 0 0, axis 1 0 0, limit lower=-1.0 upper=1.0 effort=34.0 velocity=34.0
- added joint r_hip_pitch_joint: type revolute, parent pelvis, child r_hip_pitch, origin xyz=0 -0.0762 0 rpy=0 0 0, axis 0 1 0, limit lower=-3.0 upper=3.0 effort=34.0 velocity=34.0
- added joint r_hip_roll_joint: type revolute, parent r_hip_pitch, child r_hip_roll, origin xyz=-0.05715 -0.127 0 rpy=0 0 0, axis 1 0 0, limit lower=-1.0 upper=0.279253 effort=34.0 velocity=34.0
- added joint r_hip_yaw_joint: type revolute, parent r_hip_roll, child r_hip_yaw, origin xyz=0.06254 0 -0.1905 rpy=0 0 0, axis 0 0 1, limit lower=-2.5 upper=2.5 effort=34.0 velocity=34.0
- added joint r_knee_joint: type revolute, parent r_hip_yaw, child r_knee, origin xyz=0 0 -0.2286 rpy=0 0 0, axis 0 1 0, limit lower=-0.3 upper=2.0 effort=34.0 velocity=34.0
