Commit message: fixed nemo4b

File: src/prairie_control/urdf/nemo4b.urdf (robot description, URDF)
Before this commit: robot nemo4b, 13 links, 12 joints
Links:
- link l_foot_roll: geometry collision box size=0.1 0.0505 0.006; visual mesh filename=package://prairie_control/meshes/nemo4b/l_foot_roll.stl
- link r_hip_pitch: geometry visual mesh filename=package://prairie_control/meshes/nemo4b/l_hip_pitch.stl
- link r_hip_roll: geometry visual mesh filename=package://prairie_control/meshes/nemo4b/l_hip_roll.stl
- link r_hip_yaw: geometry visual mesh filename=package://prairie_control/meshes/nemo4b/l_hip_yaw.stl
Joints:
- joint l_foot_pitch: origin xyz=0.0 0.0 0.0 rpy=0.0 0.0 0.0 -> xyz=0.0 0.0 -0.206 rpy=0 0 0
- joint l_foot_roll: origin xyz=0.0 0.0 0.0 rpy=0.0 0.0 0.0 -> xyz=0.07875 0.0 0.0 rpy=0 0 0
- joint l_hip_roll: origin xyz=0.0 0.0 0.0 rpy=0.0 0.0 0.0 -> xyz=-0.07875 0.0 0.0 rpy=0 0 0
- joint l_hip_yaw: limit lower=-1.0 upper=1.0 effort=100 velocity=100 -> lower=-1.0 upper=1.0 effort=46 velocity=100; origin xyz=0.0 0.0 0.0 rpy=0.0 0.0 0.0 -> xyz=0.00715 0.0 -0.1263 rpy=0 0 0
- joint l_knee: origin xyz=0.0 0.0 0.0 rpy=0.0 0.0 0.0 -> xyz=0.0 0.0 -0.07875 rpy=0 0 0
- joint r_foot_pitch: origin xyz=0.0 0.0 0.0 rpy=0.0 0.0 0.0 -> xyz=0.0 0.0 -0.206 rpy=0 0 0
- joint r_foot_roll: origin xyz=0.0 0.0 0.0 rpy=0.0 0.0 0.0 -> xyz=0.07875 0.0 0.0 rpy=0 0 0
- joint r_hip_roll: origin xyz=0.0 0.0 0.0 rpy=0.0 0.0 0.0 -> xyz=-0.07875 0.0 0.0 rpy=0 0 0
- joint r_hip_yaw: origin xyz=0.0 0.0 0.0 rpy=0.0 0.0 0.0 -> xyz=0.00715 0.0 -0.1263 rpy=0 0 0
- joint r_knee: origin xyz=0.0 0.0 0.0 rpy=0.0 0.0 0.0 -> xyz=0.0 0.0 -0.07875 rpy=0 0 0

Commit message: fixed ignore

File: src/prairie_control/urdf/nemo4b.urdf (robot description, URDF)
Before this commit: robot nemo4b, 13 links, 12 joints
Joints:
- joint l_foot_pitch: limit lower=-2.0 upper=2.0 effort=100 velocity=100 -> lower=-2.0 upper=2.0 effort=47.4 velocity=32
- joint l_foot_roll: limit lower=-1.0 upper=1.0 effort=100 velocity=100 -> lower=-1.0 upper=1.0 effort=23.7 velocity=32
- joint l_hip_pitch: limit lower=-1.3 upper=1.3 effort=100 velocity=100 -> lower=-1.3 upper=1.3 effort=47.4 velocity=32
- joint l_hip_roll: limit lower=-0.4 upper=1.5 effort=100 velocity=100 -> lower=-0.4 upper=1.5 effort=23.7 velocity=32
- joint l_hip_yaw: limit lower=-1.0 upper=1.0 effort=46 velocity=100 -> lower=-1.0 upper=1.0 effort=23.7 velocity=32
- joint l_knee: limit lower=-2.0 upper=2.0 effort=100 velocity=100 -> lower=-2.0 upper=2.0 effort=47.4 velocity=32
- joint r_foot_pitch: limit lower=-2.0 upper=2.0 effort=100 velocity=100 -> lower=-2.0 upper=2.0 effort=47.4 velocity=32
- joint r_foot_roll: limit lower=-1.0 upper=1.0 effort=100 velocity=100 -> lower=-1.0 upper=1.0 effort=23.7 velocity=32
- joint r_hip_pitch: limit lower=-1.3 upper=1.3 effort=100 velocity=100 -> lower=-1.3 upper=1.3 effort=47.4 velocity=32
- joint r_hip_roll: limit lower=-1.5 upper=0.4 effort=100 velocity=100 -> lower=-1.5 upper=0.4 effort=23.7 velocity=32
- joint r_hip_yaw: limit lower=-1.0 upper=1.0 effort=100 velocity=100 -> lower=-1.0 upper=1.0 effort=23.7 velocity=32

Commit message: stand pd

File: src/prairie_control/urdf/nemo4b.urdf (robot description, URDF)
Before this commit: robot nemo4b, 13 links, 12 joints
Links:
- link l_foot_roll: geometry collision box size=0.2 0.101 0.012; visual mesh filename=package://prairie_control/meshes/nemo4b/l_foot_roll.stl
- link r_foot_roll: geometry collision box size=0.2 0.101 0.012; visual mesh filename=package://prairie_control/meshes/nemo4b/l_foot_roll.stl
Joints:
- removed joint l_foot_pitch
- removed joint l_foot_roll
- removed joint l_hip_pitch
- removed joint l_hip_roll
- removed joint l_hip_yaw
- removed joint l_knee
- removed joint r_foot_pitch
- removed joint r_foot_roll
- removed joint r_hip_pitch
- removed joint r_hip_roll
- removed joint r_hip_yaw
- removed joint r_knee
- added joint l_foot_pitch_joint: type revolute, parent l_knee, child l_foot_pitch, origin xyz=0.0 0.0 -0.206 rpy=0 0 0, axis 0.0 1.0 0.0, limit lower=-2.0 upper=2.0 effort=47.4 velocity=32
- added joint l_foot_roll_joint: type revolute, parent l_foot_pitch, child l_foot_roll, origin xyz=0.07875 0.0 0.0 rpy=0 0 0, axis 1.0 0.0 0.0, limit lower=-1.0 upper=1.0 effort=23.7 velocity=32
- added joint l_hip_pitch_joint: type revolute, parent pelvis, child l_hip_pitch, origin xyz=0.0 0.0965 -0.112 rpy=0 0 0, axis 0.0 1.0 0.0, limit lower=-1.3 upper=1.3 effort=47.4 velocity=32
- added joint l_hip_roll_joint: type revolute, parent l_hip_pitch, child l_hip_roll, origin xyz=-0.07875 0.0 0.0 rpy=0 0 0, axis 1.0 0.0 0.0, limit lower=-0.4 upper=1.5 effort=23.7 velocity=32
- added joint l_hip_yaw_joint: type revolute, parent l_hip_roll, child l_hip_yaw, origin xyz=0.00715 0.0 -0.1263 rpy=0 0 0, axis 0.0 0.0 1.0, limit lower=-1.0 upper=1.0 effort=23.7 velocity=32
- added joint l_knee_joint: type revolute, parent l_hip_yaw, child l_knee, origin xyz=0.0 0.0 -0.07875 rpy=0 0 0, axis 0.0 1.0 0.0, limit lower=-2.0 upper=2.0 effort=47.4 velocity=32
- added joint r_foot_pitch_joint: type revolute, parent r_knee, child r_foot_pitch, origin xyz=0.0 0.0 -0.206 rpy=0 0 0, axis 0.0 1.0 0.0, limit lower=-2.0 upper=2.0 effort=47.4 velocity=32
- added joint r_foot_roll_joint: type revolute, parent r_foot_pitch, child r_foot_roll, origin xyz=0.07875 0.0 0.0 rpy=0 0 0, axis 1.0 0.0 0.0, limit lower=-1.0 upper=1.0 effort=23.7 velocity=32
- added joint r_hip_pitch_joint: type revolute, parent pelvis, child r_hip_pitch, origin xyz=0.0 -0.0965 -0.112 rpy=0.0 0.0 0.0, axis 0.0 1.0 0.0, limit lower=-1.3 upper=1.3 effort=47.4 velocity=32
- added joint r_hip_roll_joint: type revolute, parent r_hip_pitch, child r_hip_roll, origin xyz=-0.07875 0.0 0.0 rpy=0 0 0, axis 1.0 0.0 0.0, limit lower=-1.5 upper=0.4 effort=23.7 velocity=32
- added joint r_hip_yaw_joint: type revolute, parent r_hip_roll, child r_hip_yaw, origin xyz=0.00715 0.0 -0.1263 rpy=0 0 0, axis 0.0 0.0 1.0, limit lower=-1.0 upper=1.0 effort=23.7 velocity=32
- added joint r_knee_joint: type revolute, parent r_hip_yaw, child r_knee, origin xyz=0.0 0.0 -0.07875 rpy=0 0 0, axis 0.0 1.0 0.0, limit lower=-2.0 upper=2.0 effort=100 velocity=100

Commit message: working gz walk

File: src/prairie_control/urdf/nemo4b.urdf (robot description, URDF)
Before this commit: robot nemo4b, 13 links, 12 joints
Joints:
- joint r_knee_joint: limit lower=-2.0 upper=2.0 effort=100 velocity=100 -> lower=-2.0 upper=2.0 effort=47.4 velocity=32
